File: Tayloe-Mixer-v3.kicad_pcb (KiCad board)
At the start: 2 copper layers, 109 x 76.5 mm, 61 parts, among them J1 BNC, J101 Audio_Jack, J2 Conn_01x04, J3 Pad, J4 Conn_01x07_Female, J5 Pad, Q1 2N3904-SMD, Q2 2N3904-SMD, SW1 SW_DIP_x01, SW2 Rotary_Encoder_Switch, T1 6:31, T2 31:6, T3 T50_SPLITTER, U1 ESP32-A1S, U2 FST3253, U201 MAR6, U3 LM4562, U4 si5351, U5 L7805, U7 AMS1117CD-3.3

Commit message: added gerber
Other:
- board size 109 x 76.5 mm -> 112 x 78.5 mm
Changed lines of the file:
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@@
   )
   (setup
-    (last_trace_width 1)
+    (last_trace_width 0.25)
     (user_trace_width 0.5)
     (user_trace_width 0.75)
@@
     )
   )
-  (gr_line (start 155.5 26) (end 155.5 102.5) (layer Edge.Cuts) (width 0.1))
-  (gr_line (start 46.5 26) (end 155.5 26) (layer Edge.Cuts) (width 0.1))
-  (gr_line (start 46.5 102.5) (end 46.5 26) (layer Edge.Cuts) (width 0.1))
-  (gr_line (start 155.5 102.5) (end 46.5 102.5) (layer Edge.Cuts) (width 0.1))
+  (gr_line (start 156.5 25) (end 156.5 103.5) (layer Edge.Cuts) (width 0.1))
+  (gr_line (start 44.5 25) (end 156.5 25) (layer Edge.Cuts) (width 0.1))
+  (gr_line (start 44.5 103.5) (end 44.5 25) (layer Edge.Cuts) (width 0.1))
+  (gr_line (start 156.5 103.5) (end 44.5 103.5) (layer Edge.Cuts) (width 0.1))
   (segment (start 140.8 85.025) (end 147.1 85.025) (width 1) (layer F.Cu) (net 1))
   (via (at 129.5 84) (size 1.2) (drill 0.4) (layers F.Cu B.Cu) (net 1))
@@
     (polygon
       (pts
-        (xy 155.5 102.5) (xy 46.5 102.5) (xy 46.5 26.5) (xy 155.5 26.5)
+        (xy 156 103) (xy 45 103) (xy 45 25.5) (xy 156 25.5)
       )
     )
@@
     (polygon
       (pts
-        (xy 155 102.5) (xy 47 102.5) (xy 47 26.5) (xy 155 26.5)
+        (xy 156 103) (xy 45 103) (xy 45 25.5) (xy 156 25.5)
       )
     )
